File: PCB/MP3_Player.kicad_pcb (KiCad board)
At the start: 2 copper layers, 47.4 x 68.9 mm, 16 parts, among them J1 Micro_SD_Card_Det2, J2 Conn_01x04_Pin, J3 Conn_01x04_Pin, J5 Conn_01x05_Socket, U1 ESP32-WROVER-E, U3 CH340C

Commit message: Change
Routing:
- added copper zone on B.Cu, net Earth
- added copper zone on F.Cu, net Earth
Other:
- outline, holes or cut-outs redrawn
Changed lines of the file:
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@@
 			(outputformat 1)
 			(mirror no)
-			(drillshape 1)
+			(drillshape 0)
 			(scaleselection 1)
-			(outputdirectory "")
+			(outputdirectory "C:/Users/Adiptoo/Downloads/W/")
 		)
 	)
@@
 		(at 132.045 52.89 -90)
 		(property "Reference" "U3"
-			(at -0.48 -6.885 90)
+			(at -0.49 -6.345 90)
 			(layer "F.SilkS")
 			(effects
@@
 			(at 0 -1.68 0)
 			(layer "F.SilkS")
+			(hide yes)
 			(effects
 				(font
@@
 			(at 0 1.68 0)
 			(layer "F.Fab")
+			(hide yes)
 			(effects
 				(font
@@
 			(at 0 5.505 90)
 			(layer "F.Fab")
+			(hide yes)
 			(effects
 				(font
@@
 			(at 0 -1.68 0)
 			(layer "F.SilkS")
+			(hide yes)
 			(effects
 				(font
@@
 			(at 0 1.68 0)
 			(layer "F.Fab")
+			(hide yes)
 			(effects
 				(font
@@
 		(tags "esp32 module")
 		(property "Reference" "U1"
-			(at -0.14 -17.145 0)
+			(at -12.49 -13.275 0)
 			(layer "F.SilkS")
 			(effects
@@
 		)
 		(fp_text user "${REFERENCE}"
-			(at 0 0 0)
+			(at 1.42 -1.865 0)
 			(layer "F.Fab")
 			(effects
@@
 			(at 1.375 1.5 0)
 			(layer "B.SilkS")
+			(hide yes)
 			(effects
 				(font
@@
 		)
 	)
-	(gr_rect
-		(start 91.8 44.22)
-		(end 139.2 113.12)
+	(gr_arc
+		(start 92.8 113.12)
+		(mid 92.092893 112.827107)
+		(end 91.8 112.12)
+		(stroke
+			(width 0.05)
+			(type default)
+		)
+		(layer "Edge.Cuts")
+	)
+	(gr_arc
+		(start 91.8 45.22)
+		(mid 92.092893 44.512893)
+		(end 92.8 44.22)
+		(stroke
+			(width 0.05)
+			(type default)
+		)
+		(layer "Edge.Cuts")
+	)
+	(gr_arc
+		(start 139.2 112.12)
+		(mid 138.907107 112.827107)
+		(end 138.2 113.12)
+		(stroke
+			(width 0.05)
+			(type default)
+		)
+		(layer "Edge.Cuts")
+	)
+	(gr_arc
+		(start 138.2 44.22)
+		(mid 138.907107 44.512893)
+		(end 139.2 45.22)
+		(stroke
+			(width 0.05)
+			(type default)
+		)
+		(layer "Edge.Cuts")
+	)
+	(gr_line
+		(start 139.2 45.22)
+		(end 139.2 112.12)
+		(stroke
+			(width 0.05)
+			(type default)
+		)
+		(layer "Edge.Cuts")
+	)
+	(gr_line
+		(start 91.8 112.12)
+		(end 91.8 45.22)
+		(stroke
+			(width 0.05)
+			(type default)
+		)
+		(layer "Edge.Cuts")
+	)
+	(gr_line
+		(start 138.2 113.12)
+		(end 92.8 113.12)
+		(stroke
+			(width 0.05)
+			(type default)
+		)
+		(layer "Edge.Cuts")
+	)
+	(gr_line
+		(start 92.8 44.22)
+		(end 138.2 44.22)
 		(stroke
 			(width 0.05)
 			(type default)
 		)
-		(fill no)
 		(layer "Edge.Cuts")
 	)
@@
 	)
 	(segment
+		(start 136.49 50.794999)
+		(end 136.49 50.14)
+		(width 0.2)
+		(layer "F.Cu")
+		(net 2)
+	)
+	(segment
 		(start 126.819 45.421)
 		(end 127.16 45.08)
@@
 	)
 	(segment
-		(start 136.49 50.794999)
-		(end 136.49 50.14)
+		(start 129.18 45.08)
+		(end 130.16 46.06)
 		(width 0.2)
 		(layer "F.Cu")
@@
 	)
 	(segment
-		(start 129.18 45.08)
-		(end 130.16 46.06)
+		(start 133.339 59.311)
+		(end 133.339 53.945999)
 		(width 0.2)
 		(layer "F.Cu")
@@
 	)
 	(segment
-		(start 133.339 58.681)
-		(end 133.339 53.945999)
-		(width 0.2)
-		(layer "F.Cu")
-		(net 2)
-	)
-	(segment
 		(start 136.49 48.86)
 		(end 136.49 50.14)
@@
 	)
 	(segment
+		(start 133.339 53.945999)
+		(end 136.49 50.794999)
+		(width 0.2)
+		(layer "F.Cu")
+		(net 2)
+	)
+	(segment
 		(start 135.79 48.16)
 		(end 136.49 48.86)
@@
 	)
 	(segment
+		(start 132.38 60.27)
+		(end 133.339 59.311)
+		(width 0.2)
+		(layer "F.Cu")
+		(net 2)
+	)
+	(segment
+		(start 131.75 60.27)
+		(end 132.38 60.27)
+		(width 0.2)
+		(layer "F.Cu")
+		(net 2)
+	)
+	(segment
 		(start 106.73 52.5)
 		(end 107.68 52.5)
@@
 	)
 	(segment
-		(start 131.75 60.27)
-		(end 133.339 58.681)
-		(width 0.2)
-		(layer "F.Cu")
-		(net 2)
-	)
-	(segment
-		(start 133.339 53.945999)
-		(end 136.49 50.794999)
-		(width 0.2)
-		(layer "F.Cu")
-		(net 2)
-	)
-	(segment
 		(start 102.21 95.45)
 		(end 101.43 96.23)
@@
 	)
 	(segment
-		(start 123.26 90.72)
-		(end 120.78 93.2)
+		(start 132.476 59.696)
+		(end 132.476 72.504)
+		(width 0.2)
+		(layer "B.Cu")
+		(net 4)
+	)
+	(segment
+		(start 132.05 59.27)
+		(end 132.476 59.696)
 		(width 0.2)
 		(layer "B.Cu")
@@
 	)
 	(segment
+		(start 123.26 90.72)
+		(end 120.78 93.2)
+		(width 0.2)
+		(layer "B.Cu")
+		(net 4)
+	)
+	(segment
 		(start 131.77672 59.27)
-		(end 132.476 59.96928)
+		(end 132.05 59.27)
 		(width 0.2)
 		(layer "B.Cu")
@@
 	)
 	(segment
-		(start 126.65 78.33)
-		(end 132.476 72.504)
+		(start 126.65 85.22)
+		(end 123.26 88.61)
 		(width 0.2)
 		(layer "B.Cu")
@@
 	)
 	(segment
-		(start 136.49 55.64)
-		(end 136.49 53.95)
+		(start 123.26 88.61)
+		(end 123.26 90.72)
 		(width 0.2)
 		(layer "B.Cu")
@@
 	)
 	(segment
-		(start 132.476 59.96928)
-		(end 132.476 72.504)
+		(start 136.49 55.64)
+		(end 136.49 53.95)
 		(width 0.2)
 		(layer "B.Cu")
@@
 	)
 	(segment
-		(start 123.26 88.61)
-		(end 123.26 90.72)
+		(start 132.476 72.504)
+		(end 126.65 78.33)
 		(width 0.2)
 		(layer "B.Cu")
@@
 	)
 	(segment
-		(start 126.65 85.22)
-		(end 123.26 88.61)
+		(start 131.75 57.06)
+		(end 131.75 59.27)
 		(width 0.2)
 		(layer "B.Cu")
@@
 	)
 	(segment
-		(start 131.75 57.06)
-		(end 131.75 59.27)
-		(width 0.2)
-		(layer "B.Cu")
-		(net 4)
-	)
-	(segment
 		(start 121.28 63.39)
 		(end 121.28 75.85)
@@
 	)
 	(segment
+		(start 118.42 73)
+		(end 118.37 73.05)
+		(width 0.2)
+		(layer "F.Cu")
+		(net 7)
+	)
+	(segment
 		(start 123.28 62.66)
 		(end 122.06 63.88)
@@
 	)
 	(segment
-		(start 118.42 73)
-		(end 118.37 73.05)
+		(start 118.865 69.835)
+		(end 118.42 70.28)
 		(width 0.2)
 		(layer "F.Cu")
@@
 	)
 	(via
-		(at 118.42 70.28)
+		(at 118.865 69.835)
 		(size 0.6)
 		(drill 0.3)
@@
 	(segment
 		(start 121.12 67.58)
-		(end 118.42 70.28)
+		(end 118.865 69.835)
 		(width 0.2)
 		(layer "B.Cu")
@@
 	)
 	(segment
-		(start 130.950999 58.024)
-		(end 128.366 58.024)
+		(start 131.114999 57.86)
+		(end 128.53 57.86)
 		(width 0.2)
 		(layer "F.Cu")
@@
 	(segment
 		(start 132.68 56.294999)
-		(end 130.950999 58.024)
+		(end 131.114999 57.86)
 		(width 0.2)
 		(layer "F.Cu")
@@
 	)
 	(segment
-		(start 128.366 58.024)
-		(end 127.34 59.05)
+		(start 132.68 55.64)
+		(end 132.68 56.294999)
 		(width 0.2)
 		(layer "F.Cu")
@@
 	)
 	(segment
-		(start 132.68 55.64)
-		(end 132.68 56.294999)
+		(start 128.53 57.86)
+		(end 127.34 59.05)
 		(width 0.2)
 		(layer "F.Cu")
@@
 	)
 	(segment
-		(start 133.95 61.919942)
-		(end 133.95 55.64)
+		(start 130.86 65.38)
+		(end 133.95 62.29)
 		(width 0.2)
 		(layer "F.Cu")
@@
 	(segment
 		(start 128.098527 65.38)
-		(end 130.489942 65.38)
+		(end 130.86 65.38)
 		(width 0.2)
 		(layer "F.Cu")
@@
 	)
 	(segment
-		(start 130.489942 65.38)
-		(end 133.95 61.919942)
+		(start 133.95 62.29)
+		(end 133.95 55.64)
 		(width 0.2)
 		(layer "F.Cu")
@@
 		(net 52)
 	)
+	(zone
+		(net 2)
+		(net_name "Earth")
+		(layers "F.Cu" "B.Cu")
+		(hatch edge 0.5)
+		(connect_pads
+			(clearance 0.5)
+		)
+		(min_thickness 0.25)
+		(filled_areas_thickness no)
+		(fill yes
+			(thermal_gap 0.5)
+			(thermal_bridge_width 0.5)
+		)
+		(polygon
+			(pts
+				(xy 105.46 44.27) (xy 92.72 44.22) (xy 92.24 44.36) (xy 91.94 44.73) (xy 91.81 45.03) (xy 91.8 45.38)
+				(xy 91.8 112.1) (xy 91.84 112.44) (xy 92.06 112.8) (xy 92.49 113.08) (xy 92.96 113.12) (xy 138.22 113.12)
+				(xy 138.71 112.98) (xy 139.06 112.64) (xy 139.2 112.18) (xy 139.2 45.22) (xy 139.11 44.79) (xy 138.84 44.46)
+				(xy 138.48 44.24) (xy 138.02 44.21) (xy 125.48 44.22) (xy 125.5 51.81) (xy 105.49 51.58)
+			)
+		)
+	)
 	(embedded_fonts no)
