File: PCB/MP3_Player.kicad_sch (KiCad schematic)
At the start: 16 parts, among them J1 Micro_SD_Card_Det2, J2 Conn_01x04_Pin, J3 Conn_01x04_Pin, J5 Conn_01x05_Socket, U1 ESP32-WROVER-E, U3 CH340C

Commit message: Change
Other:
- moved on the sheet: J1
Changed lines of the file:
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@@
 	(wire
 		(pts
-			(xy 102.87 50.8) (xy 116.84 50.8)
+			(xy 102.87 50.8) (xy 140.97 50.8)
 		)
 		(stroke
@@
 	(wire
 		(pts
-			(xy 116.84 50.8) (xy 116.84 53.34)
-		)
-		(stroke
-			(width 0)
-			(type default)
-		)
-	)
-	(wire
-		(pts
 			(xy 264.16 55.88) (xy 276.86 55.88)
 		)
@@
 	(wire
 		(pts
-			(xy 116.84 53.34) (xy 140.97 53.34)
-		)
-		(stroke
-			(width 0)
-			(type default)
-		)
-	)
-	(wire
-		(pts
 			(xy 276.86 41.91) (xy 276.86 46.99)
 		)
@@
 	(global_label "MISO"
 		(shape input)
-		(at 140.97 66.04 180)
+		(at 140.97 63.5 180)
 		(fields_autoplaced yes)
 		(effects
@@
 		)
 		(property "Intersheetrefs" "${INTERSHEET_REFS}"
-			(at 133.3886 66.04 0)
+			(at 133.3886 63.5 0)
 			(effects
 				(font
@@
 	(global_label "SCK"
 		(shape input)
-		(at 140.97 60.96 180)
+		(at 140.97 58.42 180)
 		(fields_autoplaced yes)
 		(effects
@@
 		)
 		(property "Intersheetrefs" "${INTERSHEET_REFS}"
-			(at 134.2353 60.96 0)
+			(at 134.2353 58.42 0)
 			(effects
 				(font
@@
 	(global_label "MOSI"
 		(shape input)
-		(at 140.97 55.88 180)
+		(at 140.97 53.34 180)
 		(fields_autoplaced yes)
 		(effects
@@
 		)
 		(property "Intersheetrefs" "${INTERSHEET_REFS}"
-			(at 133.3886 55.88 0)
+			(at 133.3886 53.34 0)
 			(effects
 				(font
@@
 	(symbol
 		(lib_id "power:+3.3V")
-		(at 140.97 58.42 90)
+		(at 140.97 55.88 90)
 		(unit 1)
 		(exclude_from_sim no)
@@
 		(fields_autoplaced yes)
 		(property "Reference" "#PWR06"
-			(at 144.78 58.42 0)
+			(at 144.78 55.88 0)
 			(effects
 				(font
@@
 		)
 		(property "Value" "+3.3V"
-			(at 137.16 58.4199 90)
+			(at 137.16 55.8799 90)
 			(effects
 				(font
@@
 		)
 		(property "Footprint" ""
-			(at 140.97 58.42 0)
+			(at 140.97 55.88 0)
 			(effects
 				(font
@@
 		)
 		(property "Datasheet" ""
-			(at 140.97 58.42 0)
+			(at 140.97 55.88 0)
 			(effects
 				(font
@@
 		)
 		(property "Description" "Power symbol creates a global label with name \"+3.3V\""
-			(at 140.97 58.42 0)
+			(at 140.97 55.88 0)
 			(effects
 				(font
@@
 	(symbol
 		(lib_id "power:Earth")
-		(at 140.97 63.5 270)
+		(at 140.97 60.96 270)
 		(unit 1)
 		(exclude_from_sim no)
@@
 		(fields_autoplaced yes)
 		(property "Reference" "#PWR03"
-			(at 134.62 63.5 0)
+			(at 134.62 60.96 0)
 			(effects
 				(font
@@
 		)
 		(property "Value" "Earth"
-			(at 137.16 63.4999 90)
+			(at 137.16 60.9599 90)
 			(effects
 				(font
@@
 		)
 		(property "Footprint" ""
-			(at 140.97 63.5 0)
+			(at 140.97 60.96 0)
 			(effects
 				(font
@@
 		)
 		(property "Datasheet" "~"
-			(at 140.97 63.5 0)
+			(at 140.97 60.96 0)
 			(effects
 				(font
@@
 		)
 		(property "Description" "Power symbol creates a global label with name \"Earth\""
-			(at 140.97 63.5 0)
+			(at 140.97 60.96 0)
 			(effects
 				(font
@@
 	(symbol
 		(lib_id "power:Earth")
-		(at 184.15 73.66 0)
+		(at 184.15 71.12 0)
 		(unit 1)
 		(exclude_from_sim no)
@@
 		(fields_autoplaced yes)
 		(property "Reference" "#PWR01"
-			(at 184.15 80.01 0)
+			(at 184.15 77.47 0)
 			(effects
 				(font
@@
 		)
 		(property "Value" "Earth"
-			(at 184.15 78.74 0)
+			(at 184.15 76.2 0)
 			(effects
 				(font
@@
 		)
 		(property "Footprint" ""
-			(at 184.15 73.66 0)
+			(at 184.15 71.12 0)
 			(effects
 				(font
@@
 		)
 		(property "Datasheet" "~"
-			(at 184.15 73.66 0)
+			(at 184.15 71.12 0)
 			(effects
 				(font
@@
 		)
 		(property "Description" "Power symbol creates a global label with name \"Earth\""
-			(at 184.15 73.66 0)
+			(at 184.15 71.12 0)
 			(effects
 				(font
@@
 	(symbol
 		(lib_id "Connector:Micro_SD_Card_Det2")
-		(at 163.83 60.96 0)
+		(at 163.83 58.42 0)
 		(unit 1)
 		(exclude_from_sim no)
@@
 		(fields_autoplaced yes)
 		(property "Reference" "J1"
-			(at 164.465 39.37 0)
+			(at 164.465 36.83 0)
 			(effects
 				(font
@@
 		)
 		(property "Value" "Micro_SD_Card_Det2"
-			(at 164.465 41.91 0)
+			(at 164.465 39.37 0)
 			(effects
 				(font
@@
 		)
 		(property "Footprint" "Connector_Card:microSD_HC_Hirose_DM3AT-SF-PEJM5"
-			(at 215.9 43.18 0)
+			(at 215.9 40.64 0)
 			(effects
 				(font
@@
 		)
 		(property "Datasheet" "https://www.hirose.com/en/product/document?clcode=&productname=&series=DM3&documenttype=Catalog&lang=en&documentid=D49662_en"
-			(at 166.37 58.42 0)
+			(at 166.37 55.88 0)
 			(effects
 				(font
@@
 		)
 		(property "Description" "Micro SD Card Socket with two card detection pins"
-			(at 163.83 60.96 0)
+			(at 163.83 58.42 0)
 			(effects
 				(font
